File: STEMBoT-2 UEXT Modules/All Modules.sch (EAGLE design)
At the start: 53 parts, among them IC3 8to3 Encoder, IC6 8to3 Encoder, U1 HC-SR04, U2 TESEO-LIV3F, U3 CYBLE-012011-00

Commit message: changes to pcb with 6 mil traces
Parts:
- removed IC3, IC6: 8to3 Encoder, 74xx-eu:74LS348FK
- removed R10, R11, R12, R13, R14, R9: 10k, ngspice-simulation:R
- removed UX1, UX2, UX3, UX4, UX5, UX8, UX9: UEXT-CON, UEXT-Connecotr:UEXT-CON
- added R23, R24, R25, R26, R27, R28, R29, R30: 10k, rcl:R-EU_M1206
- added U$12, U$2, U$3, U$7, U$8: UEXT-SMD, UEXT-Connecotr:UEXT-SMD
- added U$13, U$14: PARALLEL2SERIAL, SOIC127P600X175-16N:PARALLEL2SERIAL
- R17, R18, R19, R2, R20, R21, R3, R8: device ngspice-simulation:R -> rcl:R-EU_M1206
- U$5, U$9: value LPC11C24FBD48/301 -> UEXT-SMD; device QFP50P900X900X160-48N:LPC11C24FBD48/301 -> UEXT-Connecotr:UEXT-SMD
Connections:
- removed net N$46: IC3A.A1, U$5.R/PIO1_1/AD2/CT32B1_MAT0
- removed net N$47: IC3A.A2, U$5.R/PIO1_2/AD3/CT32B1_MAT1
- removed net N$70: U$9.PIO1_6/RXD/CT32B0_MAT0, UX8.TXD
- removed net N$71: U$9.PIO1_7/TXD/CT32B0_MAT1, UX8.RXD
- removed net N$72: IC6A.A0, U$9.R/PIO1_0/AD1/CT32B1_CAP0
- removed net N$73: IC6A.A1, U$9.R/PIO1_1/AD2/CT32B1_MAT0
- removed net N$74: IC6A.A2, U$9.R/PIO1_2/AD3/CT32B1_MAT1
- new net N$18: PHOTORESISTOR1.1, R24.1
- new net N$20: R16.1E, R8.1
- net N$1: now also U$8.3.3V; no longer UX2.3.3V
- net N$10: now also IC1P.V+, IC2P.V+, R21.2, U$13.D7, U$13.VCC, U$2.GND; no longer IC3A.7, IC3A.EI, R14.1, U$5.GND, U$5.RESET/PIO0_0, UX1.GND
- net N$11: now also U$13.DS, U$2.SCK; no longer U$5.PIO1_7/TXD/CT32B0_MAT1, UX1.RXD
- net N$12: now also U$14.Q, U$3.RXD; no longer IC3A.A0, U$5.R/PIO1_0/AD1/CT32B1_CAP0
- net N$14: now also U$5.GND; no longer UX3.GND
- net N$15: now also U$5.TXD; no longer UX3.TXD
- net N$16: now also U$5.RXD; no longer UX3.RXD
- net N$19: now also U$14.DS, U$3.SCK; no longer U$9.RESET/PIO0_0
- net N$21: now also U$9.GND; no longer UX5.GND
- net N$22: now also U$9.3.3V; no longer UX5.3.3V
- net N$23: now also U$9.SCL; no longer UX5.SCL
- net N$24: now also U$9.SDA; no longer UX5.SDA
- net N$26: now also U$12.3.3V; no longer UX4.3.3V
- net N$27: now also U$12.SDA; no longer UX4.SDA
- net N$28: now also U$12.SCL; no longer UX4.SCL
- net N$29: now also U$12.GND; no longer UX4.GND
- net N$3: now also U$8.GND; no longer UX2.GND
- net N$33: now also R2.2, R3.1; no longer R8.1, R9.2
- net N$34: now also R17.1, R3.2; no longer R10.2, R9.1
- net N$35: now also R17.2, R18.1; no longer R10.1, R11.2
- net N$36: now also R18.2, R19.1; no longer R11.1, R12.2
- net N$37: now also R19.2, R20.1; no longer R12.1, R13.2
- net N$38: now also R20.2, R21.1; no longer R13.1, R14.2
- net N$39: now also U$13.D0; no longer IC3A.0
- net N$4: now also U$8.TXD; no longer UX2.TXD
- net N$40: now also U$13.D1; no longer IC3A.1
- net N$41: now also U$13.D2; no longer IC3A.2
- net N$42: now also U$13.D3; no longer IC3A.3
- net N$43: now also U$13.D4; no longer IC3A.4
- net N$44: now also U$13.D5; no longer IC3A.5
- net N$45: now also U$13.D6; no longer IC3A.6
- net N$48: now also R8.2; no longer R16.1E
- net N$49: now also R25.2, R26.1; no longer R17.2, R3.1
- net N$5: now also U$8.RXD; no longer UX2.RXD
- net N$50: now also R2.1; no longer R8.2
- net N$52: now also IC1P.V-, IC2P.V-, U$13.GND, U$2.3.3V; no longer U$5.VCC, UX1.3.3V
- net N$54: now also R26.2, R27.1; no longer R17.1, R18.2
- net N$55: now also R27.2, R28.1; no longer R18.1, R19.2
- net N$56: now also R28.2, R29.1; no longer R19.1, R20.2
- net N$57: now also R29.2, R30.1; no longer R20.1, R21.2
- net N$58: now also U$14.D0; no longer IC6A.0
- net N$59: now also U$14.D1; no longer IC6A.1
- net N$60: now also U$14.D2; no longer IC6A.2
- net N$61: now also U$14.D3; no longer IC6A.3
- net N$62: now also U$14.D4; no longer IC6A.4
- net N$63: now also U$14.D5; no longer IC6A.5
- net N$64: now also U$14.D6; no longer IC6A.6
- net N$65: now also R24.2; no longer PHOTORESISTOR1.1
- net N$66: now also IC4P.V-, IC5P.V-, U$14.GND, U$3.3.3V; no longer U$9.VCC, UX8.3.3V
- net N$68: now also R23.1; no longer R2.2
- net N$69: now also IC4P.V+, IC5P.V+, R30.2, U$14.D7, U$14.VCC, U$3.GND; no longer IC6A.7, IC6A.EI, R21.1, U$9.GND, UX8.GND
- net N$7: now also U$5.3.3V; no longer UX3.3.3V
- net N$8: now also U$13.Q, U$2.RXD; no longer U$5.PIO1_6/RXD/CT32B0_MAT0, UX1.TXD
- net N$81: now also U$7.3.3V; no longer UX9.3.3V
- net N$84: now also U$7.GND; no longer UX9.GND
- net N$85: now also U$7.TXD; no longer UX9.TXD
- net N$86: now also U$7.RXD; no longer UX9.RXD
- net N$9: now also R23.2, R25.1; no longer R2.1, R3.2
Other:
- note removed: "UEXT Photo Resistor Module"
- moved on the sheet: R17, R18, R19, R2, R20, R21, R3, R8

Commit message: added changes to adc shematic design
Parts:
- removed IC2, IC4, IC5: (no value), linear:4AMP_P4+11D
- removed LED3, LED6, LED7: NFSG036BT, led:NFSG036BT
- removed PHOTORESISTOR1: M9960_11A, photo-elements:M9960_11A
- removed R20, R24, R25, R26, R27, R28, R29, R30: 10k, rcl:R-EU_M1206
- removed U$13, U$14: PARALLEL2SERIAL, SOIC127P600X175-16N:PARALLEL2SERIAL
- removed U$4: HW740, IRSensors:HW740
- removed U$5: UEXT-SMD, UEXT-Connecotr:UEXT-SMD
- added D1: SFH482, led:SFH482
- added D2: BP104, opto-trans-siemens:BP104
- added DZ1: LZR182, led:LZR182
- added IC3: 74HC165PW,118, 74HC165PW_118:74HC165PW,118
- added LED8: LSG-T676, led:LSG-T676
- added PH1: VT20N1, photo-elements:VT20N1
- added Q1: MMBT3904LP-7, NPN BJT:MMBT3904LP-7
- added Q2: MMBT3904LP-7, MMBT3904LP-7:MMBT3904LP-7
- added R10, R11, R12, R13, R14, R31, R32, R33, R34, R35, R36, R37, R38, R39, R9: ERJ-1RHD3601C, Resistor:ERJ-1RHD3601C
- added U4, U7: SN74HC148D, SN74HC148D:SN74HC148D
- added U5, U6, U8, U9: MAX964ESET, MAX964ESET:MAX964ESET
- added VR1: PVG3A200C01R00, TrimmerPot:PVG3A200C01R00
- IC1: value (none) -> 74HC165PW,118; device linear:4AMP_P4+11D -> 74HC165PW_118:74HC165PW,118
- R15, R4, R5: value 1k -> ERJ-1RHD3601C; device rcl:R-EU_M1206 -> Resistor:ERJ-1RHD3601C
- R16: value 1K ohm -> ERJ-1RHD3601C; device piher:PC16S -> Resistor:ERJ-1RHD3601C
- R17, R18, R19, R2, R21, R23, R3, R8: value 10k -> ERJ-1RHD3601C; device rcl:R-EU_M1206 -> Resistor:ERJ-1RHD3601C
- U$1: value LPC11C24FBD48/301 -> UEXT-SMD; device QFP50P900X900X160-48N:LPC11C24FBD48/301 -> UEXT-Connecotr:UEXT-SMD
Connections:
- removed net N$15: U$1.PIO1_6/RXD/CT32B0_MAT0, U$5.TXD
- removed net N$17: U$1.R/PIO0_11/AD0/CT32B0_MAT3, U$4.VOUT
- removed net N$53: LED3.C, R4.2
- removed net N$54: IC4D.-IN, R26.2, R27.1
- removed net N$56: IC5B.-IN, R28.2, R29.1
- removed net N$57: IC5C.-IN, R29.2, R30.1
- removed net N$58: IC4A.OUT, U$14.D0
- removed net N$59: IC4B.OUT, U$14.D1
- removed net N$60: IC4C.OUT, U$14.D2
- removed net N$61: IC4D.OUT, U$14.D3
- removed net N$62: IC5A.OUT, U$14.D4
- removed net N$63: IC5B.OUT, U$14.D5
- removed net N$64: IC5C.OUT, U$14.D6
- removed net N$65: IC4A.+IN, IC4B.+IN, IC4C.+IN, IC4D.+IN, IC5A.+IN, IC5B.+IN, IC5C.+IN, R24.2
- removed net N$66: IC4P.V-, IC5P.V-, R15.1, U$14.GND, U$3.3.3V
- removed net N$67: LED6.C, R15.2
- removed net N$68: IC4A.-IN, PHOTORESISTOR1.2, R23.1
- removed net N$69: IC4P.V+, IC5P.V+, LED6.A, R30.2, U$14.D7, U$14.VCC, U$3.GND
- new net N$100: U4.4, U6.QA
- new net N$101: U4.2, U6.QB
- new net N$102: U4.1, U6.QC
- new net N$103: U4.0, U6.QD
- new net N$31: D1.C, R9.2
- new net N$32: LED8A.A, R11.2
- new net N$46: LED8B.A, R12.1
- new net N$47: LED8B.C, Q1.C
- new net N$51: IC1.VCC, PH1.1, R23.1, R3.2, R8.2, U$3.3.3V, U7.VCC, U8.GND, U8.VCC
- new net N$70: D2.A, R10.2
- new net N$71: R14.1, VR1.WIPER
- new net N$72: Q1.B, R13.1
- new net N$74: IC3.D0, U4.A0
- new net N$75: IC3.D1, U4.A1
- new net N$76: IC3.D2, U4.A2
- new net N$77: IC3.Q7, R13.2, U$1.MISO
- new net N$79: R14.2, U5.INA+, U5.INB+, U5.INC+, U5.IND+, U6.INA+, U6.INB+, U6.INC+, U6.IND+
- new net N$80: R34.1, R39.2, U5.INA-
- new net N$83: R32.1, R34.2, U5.INB-
- new net N$89: R32.2, R35.1, U5.INC-
- new net N$91: R31.1, R35.2, U5.IND-
- new net N$92: R31.2, R36.2, U6.INA-
- new net N$93: R33.2, R36.1, U6.INB-
- new net N$94: R33.1, R37.2, U6.INC-
- new net N$95: R37.1, R38.2, U6.IND-
- new net N$96: U4.7, U5.QA
- new net N$97: U4.6, U5.QB
- new net N$98: U4.5, U5.QC
- new net N$99: U4.3, U5.QD
- net N$10: now also DZ1-2.C, Q2.C; no longer IC1P.V+, IC2P.V+, LED3.A, R21.2, U$13.D7, U$13.VCC, U$2.GND
- net N$11: now also IC1.D2, U7.A2; no longer U$13.DS, U$2.SCK
- net N$12: now also PH1.2, R5.1, U8.INA+, U8.INB+, U8.INC+, U8.IND+, U9.INA+, U9.INB+, U9.INC+, U9.IND+; no longer U$14.Q, U$3.RXD
- net N$13: now also IC1.!CE, U$3.SSEL; no longer LED7.A, R5.2
- net N$14: now also IC3.CP, U$1.SCK; no longer LED7.C, U$1.RESET/PIO0_0, U$4.VCC, U$5.GND
- net N$16: now also IC1.Q7, R4.1; no longer U$1.PIO1_7/TXD/CT32B0_MAT1, U$5.RXD
- net N$18: now also DZ1-2.A, R23.2; no longer PHOTORESISTOR1.1, R24.1
- net N$19: now also IC1.D0, U7.A0; no longer U$14.DS, U$3.SCK
- net N$20: now also IC1.D1, IC1.DS, U7.A1; no longer R16.1E, R8.1
- net N$33: now also R15.1, R2.1, U8.INB-; no longer IC1B.-IN, R2.2, R3.1
- net N$34: now also R15.2, R16.2, U8.INC-; no longer IC1C.-IN, R17.1, R3.2
- net N$35: now also R16.1, U8.IND-; no longer IC1D.-IN, R18.1
- net N$36: now also R17.1, R21.2, U9.INA-; no longer IC2A.-IN, R18.2, R19.1
- net N$37: now also R18.1, R21.1, U9.INB-; no longer IC2B.-IN, R19.2, R20.1
- net N$38: now also R18.2, R19.2, U9.INC-; no longer IC2C.-IN, R20.2, R21.1
- net N$39: now also DZ1-1.C, IC1.GND, Q2.E, R19.1, R5.2, U$3.GND, U7.GND, U9.GND, U9.IND-; no longer IC1A.OUT, U$13.D0
- net N$40: now also U7.7, U8.QA; no longer IC1B.OUT, U$13.D1
- net N$41: now also U7.6, U8.QB; no longer IC1C.OUT, U$13.D2
- net N$42: now also U7.5, U8.QC; no longer IC1D.OUT, U$13.D3
- net N$43: now also U7.3, U8.QD; no longer IC2A.OUT, U$13.D4
- net N$44: now also U7.4, U9.QA; no longer IC2B.OUT, U$13.D5
- net N$45: now also U7.2, U9.QB; no longer IC2C.OUT, U$13.D6
- net N$48: now also U7.1, U9.QC; no longer IC1A.+IN, IC1B.+IN, IC1C.+IN, IC1D.+IN, IC2A.+IN, IC2B.+IN, IC2C.+IN, R8.2
- net N$49: now also U7.0, U9.QD; no longer IC4C.-IN, R25.2, R26.1
- net N$50: now also R2.2, R8.1, U8.INA-; no longer IC1A.-IN, R16.1A, R16.1S, R2.1
- net N$52: now also IC1.CP, U$3.SCK; no longer IC1P.V-, IC2P.V-, R4.1, U$13.GND, U$2.3.3V
- net N$55: now also D1.A, D2.C, IC3.D3, IC3.D4, IC3.D5, IC3.D6, IC3.D7, IC3.GND, IC3.VCC, LED8A.C, Q1.E, R10.1, R11.1, R12.2, R38.1, R39.1, R9.1, U$1.3.3V, U$1.GND, U4.GND, U4.VCC, U5.GND, U5.VCC, U6.GND, U6.VCC, VR1.CCW, VR1.CW; no longer IC5A.-IN, R27.2, R28.1
- net N$7: now also IC3.!CE, U$1.SSEL; no longer R5.1, U$4.GND, U$5.3.3V
- net N$8: now also Q2.B, R4.2; no longer U$13.Q, U$2.RXD
- net N$9: now also DZ1-1.A, R3.1; no longer IC4B.-IN, R23.2, R25.1
Other:
- note added: "UEXT IR Bump Module"
- note removed: "Analog to Digital Converter Module"
- moved on the sheet: U$3

Commit message: improved schematics
Parts:
- added DZ2: LZR182, led:LZR182
- added IC2: 74HC165PW,118, 74HC165PW_118:74HC165PW,118
- added Q3: MMBT3904LP-7, MMBT3904LP-7:MMBT3904LP-7
- added R20: PC16S, piher:PC16S
- added R24, R25, R26, R27, R28, R29, R30, R40, R41, R42, R43, R44: ERJ-1RHD3601C, Resistor:ERJ-1RHD3601C
- added U10: SN74HC148D, SN74HC148D:SN74HC148D
- added U11, U12: MAX964ESET, MAX964ESET:MAX964ESET
Connections:
- new net N$104: U10.3, U11.QD
- new net N$105: U10.4, U12.QA
- new net N$106: U10.2, U12.QB
- new net N$107: U10.1, U12.QC
- new net N$108: U10.0, U12.QD
- new net N$109: R26.1, R43.2, U12.INC-
- new net N$110: R29.1, R43.1, U12.IND-
- new net N$111: DZ2-1.C, IC2.VCC, R20.1E, R20.1S, R42.2, R44.2, U10.VCC, U11.INA+, U11.INB+, U11.INC+, U11.IND+, U11.VCC, U12.INA+, U12.INB+, U12.INC+, U12.IND+, U12.VCC
- new net N$112: LED2.A, U1.VCC
- new net N$15: IC2.GND, Q3.E, R29.2, U10.EO, U10.GND, U11.GND, U12.GND
- new net N$17: IC2.D0, U10.A0
- new net N$53: IC2.D1, U10.A1
- new net N$54: IC2.D2, U10.A2
- new net N$56: R40.2
- new net N$57: DZ2-1.A, R40.1
- new net N$58: IC2.Q7, R41.2
- new net N$59: Q3.B, R41.1
- new net N$60: DZ2-2.A, R42.1
- new net N$61: DZ2-2.C, Q3.C
- new net N$62: IC2.CP
- new net N$63: R24.2, R44.1, U11.INA-
- new net N$64: R24.1, R25.1, U11.INB-
- new net N$65: R25.2, R28.1, U11.INC-
- new net N$66: R27.2, R28.2, U11.IND-
- new net N$67: R27.1, R30.2, U12.INA-
- new net N$68: R26.2, R30.1, U12.INB-
- new net N$69: U10.7, U11.QA
- new net N$73: U10.6, U11.QB
- new net N$78: U10.5, U11.QC
- net N$4: now also U$6.PIO0_5/SDA, U$8.SDA; no longer U$6.PIO1_6/RXD/CT32B0_MAT0, U$8.TXD
- net N$5: now also U$6.PIO0_4/SCL, U$8.SCL; no longer U$6.PIO1_7/TXD/CT32B0_MAT1, U$8.RXD
- net N$81: no longer U1.VCC
- net N$84: no longer LED2.A
- net N$85: now also U$10.PIO0_5/SDA, U$7.SDA; no longer U$10.PIO1_6/RXD/CT32B0_MAT0, U$7.TXD
- net N$86: now also U$10.PIO0_4/SCL, U$7.SCL; no longer U$10.PIO1_7/TXD/CT32B0_MAT1, U$7.RXD

Commit message: finished schematic
Parts:
- added C1, C10, C2, C3, C4, C5, C6, C7, C8, C9: CAPACITORS-0603, CAPACITORS:CAPACITORS-0603
- added D3: SFH482, led:SFH482
- added D4: BP104, opto-trans-siemens:BP104
- added J1, J2, J3, J4, J5, J6: FTSH-105-01-XXX-DV-K, FTSH-105-01-XXX-DV-K:FTSH-105-01-XXX-DV-K
- added LED3, LED6, LED7: NFSG036BT, led:NFSG036BT
- added PH2: VT20N1, photo-elements:VT20N1
- added R45, R46, R47, R48, R52, R53, R57, R58: 1k, rcl:R-EU_M1206
- added R49, R50, R51, R55, R61: ERJ-1RHD3601C, Resistor:ERJ-1RHD3601C
- added R54: PC16S, piher:PC16S
- added S1, S2, S3, S4, S5, S6: 2-1437565-7, 2-1437565-7 (tactile switch):2-1437565-7
- added U$13, U$15, U$5: UEXT-SMD, UEXT-Connecotr:UEXT-SMD
- added U$14, U$4: LPC11C24FBD48/301, QFP50P900X900X160-48N:LPC11C24FBD48/301
- added U13: HC-SR04, HC-SR04:HC-SR04
- added VR2: PVG3A200C01R00, TrimmerPot:PVG3A200C01R00
- R1: value 1k -> ERJ-1RHD3601C; device rcl:R-EU_M1206 -> Resistor:ERJ-1RHD3601C
- R43, R44: value ERJ-1RHD3601C -> 1k; device Resistor:ERJ-1RHD3601C -> rcl:R-EU_M1206
- U$10: value LPC11C24FBD48/301 -> UEXT-SMD; device QFP50P900X900X160-48N:LPC11C24FBD48/301 -> UEXT-Connecotr:UEXT-SMD
- U$11: value CHQ1838 -> LPC11C24FBD48/301; device IRSensors:CHQ1838 -> QFP50P900X900X160-48N:LPC11C24FBD48/301
- U$7: value UEXT-SMD -> LPC11C24FBD48/301; device UEXT-Connecotr:UEXT-SMD -> QFP50P900X900X160-48N:LPC11C24FBD48/301
- U1: value HC-SR04 -> TSL260R-LF; device HC-SR04:HC-SR04 -> TSL260R-LF:TSL260R-LF
Connections:
- removed net N$15 (its old number): IC2.GND, Q3.E, R29.2, U10.EO, U10.GND, U11.GND, U12.GND
- removed net N$3 (its old number): LED1.A, U$11.VCC, U$6.RESET/PIO0_0, U$8.GND
- removed net N$65 (its old number): R25.2, R28.1, U11.INC-
- removed net N$66 (its old number): R27.2, R28.2, U11.IND-
- removed net N$67 (its old number): R27.1, R30.2, U12.INA-
- removed net N$68 (its old number): R26.2, R30.1, U12.INB-
- new net N$105: R1.2, R42.1, U11.INA-
- new net N$106: IC2.!CE, U$2.SSEL
- new net N$107: IC2.CP, U$2.SCK
- new net N$108: IC2.VCC, R20.1E, R30.2, R40.1, R42.2, U$2.3.3V, U10.VCC, U11.GND, U11.VCC
- new net N$113: C1.2, C2.2, J1.1, LED2.A, R45.2, U$10.3.3V, U$7.VCC, U$7.VDD@44, U$7.VDD@8, U$7.VDD_CAN, U13.VCC
- new net N$114: J4.10, R48.2, S4.1, U3.XRES
- new net N$115: LED3.C, R46.2
- new net N$116: U$11.PIO0_5/SDA, U$13.SDA
- new net N$117: U$4.PIO0_5/SDA, U$5.SDA
- new net N$118: U$4.PIO0_4/SCL, U$5.SCL
- new net N$119: C3.2, C4.2, J2.1, LED3.A, R47.2, U$4.VCC, U$4.VDD@44, U$4.VDD@8, U$4.VDD_CAN, U$5.3.3V, U1.VDD
- new net N$120: J2.4, U$4.SWCLK/PIO0_10/SCK0/CT16B0_MAT2
- new net N$122: J2.2, U$4.SWDIO/PIO1_3/AD4/CT32B1_MAT2
- new net N$123: J2.6, U$4.PIO0_9/MOSI0/CT16B0_MAT1
- new net N$125: U$4.PIO2_8
- new net N$126: J4.2, U3.P0.6
- new net N$127: J2.10, R47.1, S2.3, U$4.RESET/PIO0_0
- new net N$128: J4.4, U3.P0.7
- new net N$129: J3.4, U$6.SWCLK/PIO0_10/SCK0/CT16B0_MAT2
- new net N$130: J3.2, U$6.SWDIO/PIO1_3/AD4/CT32B1_MAT2
- new net N$131: J3.6, U$6.PIO0_9/MOSI0/CT16B0_MAT1
- new net N$132: D3.C, R49.2
- new net N$133: D4.A, R50.2
- new net N$134: R51.1, VR2.WIPER
- new net N$135: J3.10, R44.1, S3.3, U$6.RESET/PIO0_0
- new net N$136: R51.2, U$6.R/PIO0_11/AD0/CT32B0_MAT3
- new net N$137: C5.1, C6.1, J3.3, J3.5, J3.9, R43.1, R49.1, R50.1, S3.2, U$6.GND, U$6.VSS@41, U$6.VSS@5, U$8.GND, VR2.CCW
- new net N$138: C5.2, C6.2, D3.A, D4.C, J3.1, LED1.A, R44.2, U$6.VCC, U$6.VDD@44, U$6.VDD@8, U$6.VDD_CAN, U$8.3.3V, VR2.CW
- new net N$139: U$11.PIO0_4/SCL, U$13.SCL
- new net N$140: J5.4, U$11.SWCLK/PIO0_10/SCK0/CT16B0_MAT2
- new net N$141: J5.2, U$11.SWDIO/PIO1_3/AD4/CT32B1_MAT2
- new net N$142: J5.6, U$11.PIO0_9/MOSI0/CT16B0_MAT1
- new net N$143: J5.10, R53.1, S5.3, U$11.RESET/PIO0_0
- new net N$144: C7.1, C8.1, J5.3, J5.5, J5.9, R52.1, R54.1A, S5.2, U$11.GND, U$11.VSS@41, U$11.VSS@5, U$13.GND
- new net N$146: R54.1S
- new net N$147: U$11.R/PIO0_11/AD0/CT32B0_MAT3
- new net N$148: C10.2, C9.2, J6.1, LED7.A, PH2.1, R58.2, U$14.VCC, U$14.VDD@44, U$14.VDD@8, U$14.VDD_CAN, U$15.3.3V
- new net N$149: C7.2, C8.2, J5.1, LED6.A, R53.2, R54.1E, U$11.VCC, U$11.VDD@44, U$11.VDD@8, U$11.VDD_CAN, U$13.3.3V
- new net N$150: LED7.C, R57.2
- new net N$151: U$14.PIO0_5/SDA, U$15.SDA
- new net N$152: U$14.PIO0_4/SCL, U$15.SCL
- new net N$153: J6.4, U$14.SWCLK/PIO0_10/SCK0/CT16B0_MAT2
- new net N$154: J6.2, U$14.SWDIO/PIO1_3/AD4/CT32B1_MAT2
- new net N$155: J6.6, U$14.PIO0_9/MOSI0/CT16B0_MAT1
- new net N$156: J6.10, R58.1, S6.3, U$14.RESET/PIO0_0
- new net N$157: PH2.2, R55.1
- new net N$159: R61.1
- new net N$160: R61.2, U$14.R/PIO0_11/AD0/CT32B0_MAT3
- new net N$161: C10.1, C9.1, J6.3, J6.5, J6.9, R55.2, R57.1, S6.2, U$14.GND, U$14.VSS@41, U$14.VSS@5, U$15.GND
- new net N$4: Q3.B, R41.2
- new net N$5: DZ2-1.A, R30.1
- new net N$61: R26.1, R29.2, U12.INA-
- new net N$82: U$10.SCL, U$7.PIO0_4/SCL
- net N$1: now also C1.1, C2.1, J1.3, J1.5, J1.9, R22.1, S1.2, U$10.GND, U$7.GND, U$7.VSS@41, U$7.VSS@5, U13.GND; no longer R1.1, U$11.GND, U$8.3.3V
- net N$109: now also R20.1S, U11.INA+, U11.INB+, U11.INC+, U11.IND+, U12.INA+, U12.INB+, U12.INC+, U12.IND+; no longer R26.1, R43.2, U12.INC-
- net N$110: now also LED6.C, R52.2; no longer R29.1, R43.1, U12.IND-
- net N$111: now also LED1.C, R43.2; no longer DZ2-1.C, IC2.VCC, R20.1E, R20.1S, R42.2, R44.2, U10.VCC, U11.INA+, U11.INB+, U11.INC+, U11.IND+, U11.VCC, U12.INA+, U12.INB+, U12.INC+, U12.IND+, U12.VCC
- net N$112: now also J1.10, R45.1, S1.3, U$7.RESET/PIO0_0; no longer LED2.A, U1.VCC
- net N$2: now also U1.OUT; no longer LED1.C, R1.2
- net N$26: now also J4.1, R48.1, S4.3
- net N$29: now also J4.3, J4.5, J4.9
- net N$53: now also IC2.DS
- net N$56: now also IC2.Q7, R41.1; no longer R40.2
- net N$57: now also DZ2-2.A, R40.2; no longer DZ2-1.A, R40.1
- net N$58: now also R1.1, R24.1, U11.INB-; no longer IC2.Q7, R41.2
- net N$59: now also R24.2, R25.2, U11.INC-; no longer Q3.B, R41.1
- net N$6: now also C3.1, C4.1, J2.3, J2.5, J2.9, R46.1, S2.2, U$4.GND, U$4.VSS@41, U$4.VSS@5, U$5.GND, U1.GND; no longer U$11.VOUT, U$6.R/PIO0_11/AD0/CT32B0_MAT3
- net N$60: now also R25.1, R26.2, U11.IND-; no longer DZ2-2.A, R42.1
- net N$62: now also R27.1, R29.1, U12.INB-; no longer IC2.CP
- net N$63: now also R27.2, R28.2, U12.INC-; no longer R24.2, R44.1, U11.INA-
- net N$64: now also DZ2-1.C, IC2.GND, Q3.E, R20.1A, R28.1, U$2.GND, U10.GND, U12.GND, U12.IND-; no longer R24.1, R25.1, U11.INB-
- net N$81: now also U$10.SDA, U$7.PIO0_5/SDA; no longer R22.1, U$7.3.3V
- net N$84: now also J1.4, U$7.SWCLK/PIO0_10/SCK0/CT16B0_MAT2; no longer U$10.RESET/PIO0_0, U$7.GND, U1.GND
- net N$85: now also J1.2, U$7.SWDIO/PIO1_3/AD4/CT32B1_MAT2; no longer U$10.PIO0_5/SDA, U$7.SDA
- net N$86: now also J1.6, U$7.PIO0_9/MOSI0/CT16B0_MAT1; no longer U$10.PIO0_4/SCL, U$7.SCL
- net N$87: now also U$7.PIO2_8, U13.TRIG; no longer U$10.R/PIO1_0/AD1/CT32B1_CAP0, U1.ECHO
- net N$88: now also U$7.PIO2_7, U13.ECHO; no longer U$10.R/PIO1_1/AD2/CT32B1_MAT0, U1.TRIG
Other:
- note added: "UEXT IR Remote Module"
- note added: "UEXT MCU IR Bump Module"
- note added: "UEXT MCU IR Photoresistor Module"
- note added: "UEXT MCU IR Potentiometer Module"
- moved on the sheet: DZ2-1, DZ2-2, IC2, LED1, LED2, Q3, R20, R22, R24, R25, R26, R27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

Commit message: added new schematic changes
Connections:
- new net N$145: IC2.!PL, U$2.MOSI
- new net N$162: IC1.!PL, U$3.MOSI
- new net N$163: IC3.!PL, U$1.MOSI
- net N$16: now also U$3.MISO
- net N$21: now also U2.GND_RF
- net N$22: now also U2.VCC_IO, U2.VCC_RF
- net N$26: now also U3.VDD, U3.VDDR, U3.VREF; no longer S4.3, U3.GND
- net N$29: now also S4.3, U3.GND; no longer U3.VDD
- net N$39: now also U7.EI
- net N$55: now also U4.EI
- net N$56: now also U$2.MISO
- net N$64: now also U10.EI
Other:
- moved on the sheet: J4, LED4, LED5, R48, R6, R7, S4, U$12, U$9, U2, U3

Commit message: removed silk screens
Parts:
- removed S4: 2-1437565-7, 2-1437565-7 (tactile switch):2-1437565-7
- added S7: B3U-1000P, B3U-1000P:B3U-1000P
- R20, R54: value PC16S -> PC16S(NOSILK); device piher:PC16S -> piher:PC16S(NOSILK)
- S1, S2, S3, S5, S6: value 2-1437565-7 -> B3U-1000P; device 2-1437565-7 (tactile switch):2-1437565-7 -> B3U-1000P:B3U-1000P
- U13: value HC-SR04 -> HC-SR04(NOSILK); device HC-SR04:HC-SR04 -> HC-SR04:HC-SR04(NOSILK)
Connections:
- net N$1: now also S6.1; no longer S1.2
- net N$112: now also S6.2; no longer S1.3
- net N$114: now also S2.1; no longer S4.1
- net N$127: now also S1.2; no longer S2.3
- net N$135: now also S7.2; no longer S3.3
- net N$137: now also S7.1; no longer S3.2
- net N$143: now also S3.2; no longer S5.3
- net N$144: now also S3.1; no longer S5.2
- net N$156: now also S5.2; no longer S6.3
- net N$161: now also S5.1; no longer S6.2
- net N$29: now also S2.2; no longer S4.3
- net N$6: now also S1.1; no longer S2.2

Commit message: changes to board and schematic
Connections:
- net N$108: now also U12.VCC
- net N$51: now also U9.VCC
Changed lines of the file:
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@@
 <junction x="-434.34" y="-132.08"/>
 <wire x1="-365.76" y1="-139.7" x2="-365.76" y2="-132.08" width="0.1524" layer="91"/>
+<pinref part="U9" gate="A" pin="VCC"/>
+<wire x1="-383.54" y1="-180.34" x2="-383.54" y2="-139.7" width="0.1524" layer="91"/>
+<junction x="-383.54" y="-139.7"/>
 </segment>
 </net>
@@
 <wire x1="-353.06" y1="38.1" x2="-353.06" y2="45.72" width="0.1524" layer="91"/>
 <pinref part="R20" gate="G$1" pin="1E"/>
-</segment>
-</net>
+<pinref part="U12" gate="A" pin="VCC"/>
+<wire x1="-370.84" y1="-2.54" x2="-370.84" y2="38.1" width="0.1524" layer="91"/>
+<junction x="-370.84" y="38.1"/>
+</segment>
+</net>
