File: STEMBoT-2 UEXT Modules/All Modules.sch (EAGLE design)
At the start: 132 parts, among them IC1 74HC165PW,118, IC2 74HC165PW,118, IC3 74HC165PW,118, J1 FTSH-105-01-XXX-DV-K, J2 FTSH-105-01-XXX-DV-K, J3 FTSH-105-01-XXX-DV-K, J4 FTSH-105-01-XXX-DV-K, J5 FTSH-105-01-XXX-DV-K, J6 FTSH-105-01-XXX-DV-K, Q1 MMBT3904LP-7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

Commit message: finish pcb traces
Parts:
- added R56, R59, R60: ERJ-1RHD3601C, Resistor:ERJ-1RHD3601C
Connections:
- removed net N$145: IC2.!PL, U$2.MOSI
- removed net N$159: R61.1
- removed net N$163: IC3.!PL, U$1.MOSI
- removed net N$2: U1.OUT
- new net N$158: IC3.!PL, R56.1, U$1.MOSI
- new net N$164: IC2.!PL, R60.1, U$2.MOSI
- net N$100: now also U4.3; no longer U4.4
- net N$125: now also U1.OUT
- net N$157: now also R61.1
- net N$162: now also R59.1
- net N$20: no longer IC1.DS
- net N$39: now also IC1.D3, IC1.D4, IC1.D5, IC1.D6, IC1.D7, R59.2
- net N$43: now also U7.4; no longer U7.3
- net N$44: now also U7.3; no longer U7.4
- net N$53: no longer IC2.DS
- net N$55: now also R56.2
- net N$64: now also IC2.D3, IC2.D4, IC2.D5, IC2.D6, IC2.D7, R60.2
- net N$68: now also U10.4; no longer U10.3
- net N$69: now also U10.3; no longer U10.4
- net N$99: now also U4.4; no longer U4.3
Other:
- moved on the sheet: R30, R61
